Commit message: WIP: more cleanup

File: modules/hopper.urdf (robot description, URDF)
Before this commit: robot hopper, 3 links, 2 joints
Links:
- link floor: geometry collision box size=2 2 0.05; collision plane normal=0 0 1
- link foot: geometry collision sphere radius=0.01; visual box size=0.05 0.05 0.05
