Commit message: new model with stick legs and much longer training

File: modules/LearningMPC/src/Models/urdf/box_atlas.urdf (robot description, URDF)
Before this commit: robot BoxAtlas, 12 links, 11 joints
Links:
- link lf: geometry collision sphere radius=0; visual cylinder length=0.45 radius=0.02
- link lf_dummy: geometry visual cylinder length=0.45 radius=0.03; visual sphere radius=0.05
- link lh: geometry collision sphere radius=0; visual cylinder length=0.375 radius=0.02
- link lh_dummy: geometry visual cylinder length=0.375 radius=0.03; visual sphere radius=0.05
- link rf: geometry collision sphere radius=0; visual cylinder length=0.45 radius=0.02
- link rf_dummy: geometry visual cylinder length=0.45 radius=0.03; visual sphere radius=0.05
- link rh: geometry collision sphere radius=0; visual cylinder length=0.375 radius=0.02
- link rh_dummy: geometry visual cylinder length=0.375 radius=0.03; visual sphere radius=0.05
Joints:
- joint core_to_lf_extension: limit lower=0.4 upper=0.9 effort=20 velocity=100 -> lower=0.45 upper=0.9 effort=20 velocity=100
- joint core_to_lh_extension: limit lower=0.18 upper=0.75 effort=2 velocity=100 -> lower=0.375 upper=0.75 effort=2 velocity=100
- joint core_to_rf_extension: limit lower=0.4 upper=0.9 effort=20 velocity=100 -> lower=0.45 upper=0.9 effort=20 velocity=100
- joint core_to_rh_extension: limit lower=0.18 upper=0.75 effort=2 velocity=100 -> lower=0.375 upper=0.75 effort=2 velocity=100
